File: PCB/nametag/nametag.kicad_pcb (KiCad board)
At the start: 2 copper layers, 45 parts, among them J1 USB_C_Receptacle_USB2.0_14P, J3 Conn_02x03_Odd_Even, Q1 NXV55UN, U1 MIC550x, U2 AVR64DU32, U3 23K640, U4 MCP9700x-ETT, U5 SN74LV1T125DBV, U6 SN74LV1T125DBV

Commit message: PCB WIP
Parts:
- added C20: 10uF, Capacitor_SMD:C_1206_3216Metric_Pad1.33x1.80mm_HandSolder, F.Cu at (207.1, 89.0)
- added C21: 10uF, Capacitor_SMD:C_1206_3216Metric_Pad1.33x1.80mm_HandSolder, F.Cu at (209.5, 89.0)
- added C22: 10uF, Capacitor_SMD:C_1206_3216Metric_Pad1.33x1.80mm_HandSolder, F.Cu at (211.9, 89.0)
- added C23: 0.1uF, 16V, Capacitor_SMD:C_0805_2012Metric_Pad1.18x1.45mm_HandSolder, F.Cu at (198.8, 84.6)
- added D4: LED, StandardPackages_Custom:LED 0805, F.Cu at (214.1, 126.3)
- added D5: LED, StandardPackages_Custom:LED 0805, F.Cu at (211.5, 126.3)
- added D6: LED, StandardPackages_Custom:LED 0805, F.Cu at (208.9, 126.3)
- added R5: 470, Resistor_SMD:R_0805_2012Metric_Pad1.20x1.40mm_HandSolder, F.Cu at (214.1, 129.8)
- added R7: 470, Resistor_SMD:R_0805_2012Metric_Pad1.20x1.40mm_HandSolder, F.Cu at (211.5, 129.8)
- added R8: 470, Resistor_SMD:R_0805_2012Metric_Pad1.20x1.40mm_HandSolder, F.Cu at (208.9, 129.8)
- added R9: 0, Resistor_SMD:R_0603_1608Metric_Pad0.98x0.95mm_HandSolder, F.Cu at (192.0, 87.7)
- R3: footprint Resistor_SMD:R_0805_2012Metric -> Resistor_SMD:R_0805_2012Metric_Pad1.20x1.40mm_HandSolder
- U4: footprint Package_TO_SOT_SMD:SOT-23 -> StandardPackages_Custom:SOT23-3
- U5, U6: footprint Package_TO_SOT_SMD:SOT-23-5 -> StandardPackages_Custom:SOT23-5
- moved C1 66.4 mm to (186.5, 93.6), turned to 0 degrees
- moved C17 65.7 mm to (205.5, 97.5)
- moved J1 64.4 mm to (183.1, 89.0)
- moved R3 64.4 mm to (187.6, 91.0)
- moved R2 64.3 mm to (187.7, 87.1)
- moved J3 63.5 mm to (205.3, 107.0), turned to 180 degrees
- moved C16 63.4 mm to (202.6, 88.5), turned to -90 degrees
- moved U1 62.5 mm to (184.5, 97.2), turned to -90 degrees
- moved C2 61.9 mm to (187.4, 97.4), turned to -90 degrees
- moved C15 60.8 mm to (199.5, 107.0), turned to -90 degrees
- moved R1 55.8 mm to (180.3, 96.4)
- moved R4 45.5 mm to (224.2, 88.3), turned to -90 degrees
- moved C6 44.7 mm to (217.4, 85.2)
- moved L1 44.5 mm to (219.9, 90.6)
- moved U3 43.5 mm to (197.1, 88.4)
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Connections:
- CLR0 pad 2: Net-(U2-PF0) -> Net-(U2-PD4)
- CLR1 pad 2: Net-(U2-PF1) -> Net-(U2-PD5)
- CLR2 pad 2: Net-(U2-PF2) -> Net-(U2-PD6)
- J1 pad S1: Net-(J1-SHIELD) -> GND
- R1 pad 1: Net-(J1-SHIELD) -> GND
- U2 pad 13: D/C -> unconnected-(U2-PD3-Pad13)
- U2 pad 14: unconnected-(U2-PD4-Pad14) -> Net-(U2-PD4)
- U2 pad 15: unconnected-(U2-PD5-Pad15) -> Net-(U2-PD5)
- U2 pad 16: unconnected-(U2-PD6-Pad16) -> Net-(U2-PD6)
- U2 pad 17: unconnected-(U2-PD7-Pad17) -> TEMP
- U2 pad 20: Net-(U2-PF0) -> LED_USB
- U2 pad 21: Net-(U2-PF1) -> LED_MEM
- U2 pad 22: Net-(U2-PF2) -> LED_DISP
- U2 pad 24: ~{DISP_RESET} -> unconnected-(U2-PF4-Pad24)
- U2 pad 25: ~{BUSY} -> unconnected-(U2-PF5-Pad25)
- U2 pad 30: unconnected-(U2-PA0-Pad30) -> D/C
- U2 pad 31: unconnected-(U2-PA1-Pad31) -> ~{DISP_RESET}
- U2 pad 32: TEMP -> ~{BUSY}
- U3 pad 3: unconnected-(U3-NC-Pad3) -> Net-(U3-NC)
Routing:
- net Net-(D1-K): track 0.00 -> 26.8 mm, vias 0 -> 2
- net SDA: track 0.00 -> 25.5 mm
- net ~{DISP_CS}: track 0.00 -> 21.4 mm, vias 0 -> 1
- net D/C: track 0.00 -> 19.9 mm
- net SCLK: track 0.00 -> 19.3 mm
- net ~{DISP_RESET}: track 0.00 -> 19.0 mm
- net ~{BUSY}: track 0.00 -> 18.9 mm
- net Net-(D1-A): track 0.00 -> 18.2 mm, vias 0 -> 2
- net GND: track 0.00 -> 15.1 mm
- net +3.3V: track 0.00 -> 14.0 mm
- net Net-(J2-RESE): track 0.00 -> 11.1 mm
- net Net-(D3-A): track 0.00 -> 10.8 mm
- net Net-(J2-VDHR): track 0.00 -> 8.56 mm
- net Net-(J2-VDDD): track 0.00 -> 7.33 mm
- net Net-(J2-VDL): track 0.00 -> 7.15 mm
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Other:
- board outline added: 59.2 x 29.2 mm
- copper layers 2 -> 4

Commit message: PCB files. BOM. Step model.
Parts:
- removed C22: 10uF, Capacitor_SMD:C_1206_3216Metric_Pad1.33x1.80mm_HandSolder
- U3: footprint StandardPackages_Custom:SOIC-8 -> Microchip:TSSOP-8 (ST)
- moved C16 30.2 mm to (186.0, 113.7)
- moved CLR2 27.0 mm to (173.1, 117.0), turned to 0 degrees
- moved CLR1 24.9 mm to (173.1, 115.5), turned to 0 degrees
- moved R5 23.8 mm to (193.9, 117.1)
- moved R7 23.8 mm to (191.3, 117.1)
- moved R8 23.8 mm to (188.7, 117.1)
- moved D4 23.8 mm to (193.9, 113.6)
- moved D5 23.8 mm to (191.3, 113.6)
- moved D6 23.8 mm to (188.7, 113.6)
- moved CLR0 22.7 mm to (173.1, 114.0), turned to 0 degrees
- moved SIZE3 20.3 mm to (173.1, 112.4), turned to 0 degrees
- moved SIZE2 18.2 mm to (173.1, 110.8), turned to 0 degrees
- moved SIZE1 16.2 mm to (173.1, 109.3), turned to 0 degrees
- moved C18 14.4 mm to (183.9, 113.7)
- moved SIZE0 14.2 mm to (173.1, 107.8), turned to 0 degrees
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Connections:
- U2 pad 1: ~{DISP_MISO_EN} -> ~{DISP_CS}
- U2 pad 23: ~{FLASH_CS} -> unconnected-(U2-PF3-Pad23)
- U2 pad 24: unconnected-(U2-PF4-Pad24) -> ~{DISP_MISO_EN}
- U2 pad 5: ~{DISP_CS} -> ~{FLASH_CS}
Routing:
- net GND: track 15.1 -> 86.1 mm, vias 0 -> 31
- net +3.3V: track 14.0 -> 76.4 mm, vias 0 -> 15
- net MOSI: track 2.10 -> 35.1 mm, vias 0 -> 4
- net MISO: track 4.95 -> 32.6 mm, vias 0 -> 2
- net SCLK: track 19.3 -> 43.3 mm, vias 0 -> 2
- net /D+: track 0.01 -> 18.9 mm
- net /D-: track 0.01 -> 18.4 mm
- net +5V: track 0.00 -> 17.3 mm
- net Net-(U2-PD6): track 0.00 -> 17.1 mm
- net Net-(U2-PD2): track 0.00 -> 17.0 mm
- net Net-(U2-PD1): track 0.00 -> 16.9 mm
- net Net-(U2-PD5): track 0.00 -> 16.8 mm
- net Net-(U2-PC3): track 0.00 -> 16.8 mm
- net Net-(U2-PD0): track 0.00 -> 16.6 mm
- net Net-(U2-PD4): track 0.00 -> 16.5 mm
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- added copper zone on In2.Cu, net +3.3V
- added copper zone on F.Cu, net GND
- added copper zone on In1.Cu, net GND
Other:
- board size 59.2 x 29.2 mm -> 61 x 31 mm
- board text added: "${REVISION}"
- board text added: "${TITLE}"
- board text added: "${TITLE} (C) Robert Perkel 2024 Revision ${REVISION} ${ISSUE_DATE}"
- board text added: "(C) Robert Perkel 2024"
- board text added: "WayWayWay"
